File: VoedingDesign_pcb/schema_pcb/schema_pcb.sch (KiCad schematic (older format))
At the start: 0 parts

Commit message: schema getekend (bijna af), nog pcb routing
Changed lines of the file:
@@
 EESchema Schematic File Version 4
+LIBS:schema_pcb-cache
 EELAYER 26 0
 EELAYER END
@@
 F0 "supercapLoader" 50
 F1 "supercapLoader.sch" 50
+F2 "output" I R 4925 4525 50
 $EndSheet
 $Sheet
@@
 F0 "BatteryLoader" 50
 F1 "BatteryLoader.sch" 50
+F2 "input" I L 5525 4525 50
 $EndSheet
-Text HLabel 5525 4525 2    50   Input ~ 0
-input
-Text HLabel 4925 4525 0    50   Input ~ 0
-output
 Wire Wire Line
 	4925 4525 5525 4525
