File: EFM32_ICM20948_PCB/Embedded_II_MAIN_BOARD.sch (EAGLE design)
At the start: 86 parts, among them IC2 EFM32HG322F64G-C-QFP48R, IC5 TPS7A0518PDBZR, Q1 20V/0.2A/8MHz/1.2Ω/1Vth, Q6 20V/0.2A/8MHz/1.2Ω/1Vth, Q8 20V/0.2A/8MHz/1.2Ω/1Vth, U3 9DoF IMU, Y2 FC-135_32.7680KA-A3, Y3 ABM3B-24.000MHZ-B2-T

Commit message: Routing main pcb
Parts:
- removed C40: 10u, microbuilder:CAP_CERAMIC0603
- added GND6, GND_1: TPTP20SQ, testpad:TPTP20SQ
- added IMU_I2C: IMU_I2C, pinhead:PINHD-1X2
- added R10, R9: 10k, microbuilder:RESISTOR0603
- added TP1, TP18, TP19, TP2, TP20, TP7, TP8, TP9: TPTP10R, testpad:TPTP10R
- renumbered JP2 to ADDR
Connections:
- net N$1 renamed IMU_VDD_PIN
- new net !CS!_RFID: IC2.PC8, RFID/SPI.4
- net !CS: no longer IC2.PC8, RFID/SPI.4
- net DBG_!RESET: now also TP9.TP
- net GND: now also GND6.TP, GND_1.TP; no longer C40.P$2
- net INT: no longer IC2.PC2
- net INT_VIN: now also IC2.PC2
- net LED: now also TP2.TP
- net LORA_EN: now also TP20.TP
- net LORA_RX: now also LORA.4, TP19.TP; no longer LORA.5
- net LORA_TX: now also LORA.5, TP18.TP; no longer LORA.4
- net PB11: no longer EXTRA.1
- net SCL: now also IMU_I2C.1, R9.1, TP8.TP
- net SDA: now also IMU_I2C.2, R10.1, TP7.TP
- net SOLAR_VOLTAGE: now also TP1.TP
- net VDD: now also R10.2, R9.2
- net V_BATT: no longer C40.P$1
Other:
- note added: "IMU I2C"
- note added: "SPI CS"
- note added: "USB Connector"
- note added: "leds"
- note removed: "USB Connector Not needed"
- moved on the sheet: C1, C21, C22, C23, TP10, TP12, TP13, TP14, TP15, U3

Commit message: main pcb lora update, bijna klaar
Parts:
- added C2, C6: 10u, rcl:C-EUC0805K
- added C3, C7: 100n, rcl:C-EUC0805K
- added C4, C5: (no value), rcl:C-EUC0603K
- added L1: WE-MK_0603_744786118, project:WE-MK_0603_744786118
- added LORA_RESET: LORA_RESET, SparkFun-Jumpers:JUMPER-SMT_2_NO_SILK
- added LORA_RX: LORA_RX, SparkFun-Jumpers:JUMPER-SMT_2_NO_SILK
- added LORA_TX: LORA_TX, SparkFun-Jumpers:JUMPER-SMT_2_NO_SILK
- added LORA_VDD: LORA_VDD, SparkFun-Jumpers:JUMPER-SMT_2_NO_SILK
- added U$2: ANTENNA868, project:ANTENNA868
- added U$4: RN2483, project:RN2483
Connections:
- new net N$1: C5.2, L1.2, U$2.P$1
- new net N$2: C4.2, L1.1, U$4.RFH
- new net N$6: LORA_RX.2, U$4.UART_RX
- new net N$7: LORA_TX.2, U$4.UART_TX
- new net N$8: LORA_RESET.2, U$4.RESET°
- new net VDD_LORA: C2.1, C3.1, C6.1, C7.1, LORA_VDD.2, U$4.VDD
- net GND: now also C2.2, C3.2, C4.1, C5.1, C6.2, C7.2, U$4.GND
- net LORA_!RESET!: now also LORA_RESET.1
- net LORA_RX: now also LORA_RX.1
- net LORA_TX: now also LORA_TX.1
- net VDD: now also LORA_VDD.1
Other:
- note added: "Lora"
- moved on the sheet: 7SEG/I2C, ANALOG, BUTTON, EXTRA, LEDS, LORA, R4, R7, R8, RFID/SPI

Commit message: finalisatie design main pcb (uC + imu + lora)
Parts:
- removed LORA: LORA, pinhead:PINHD-1X5
- removed TP20: TPTP10R, testpad:TPTP10R
- added EXTRA1: EXTRA, pinhead:PINHD-1X2
- renumbered U$4 to U4
Connections:
- removed net LORA_EN: IC2.PA8, LORA.1, TP20.TP
- removed net SENSOR_EN: IC2.PA9, LORA.2
- new net PA8: EXTRA1.1, IC2.PA8
- new net PA9: EXTRA1.2, IC2.PA9
- net LORA_!RESET!: no longer LORA.3
- net LORA_RX: no longer LORA.4
- net LORA_TX: no longer LORA.5
Changed lines of the file:
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@@
 <part name="BATT_V" library="SparkFun-Jumpers" deviceset="JUMPER-SMT_2_NO" device="_SILK" value="BATT_V"/>
 <part name="SOLAR_V" library="SparkFun-Jumpers" deviceset="JUMPER-SMT_2_NO" device="_SILK" value="SOLAR_V"/>
-<part name="LORA" library="pinhead" library_urn="urn:adsk.eagle:library:325" deviceset="PINHD-1X5" device="" package3d_urn="urn:adsk.eagle:package:22469/2" value="LORA"/>
 <part name="EXTRA" library="pinhead" library_urn="urn:adsk.eagle:library:325" deviceset="PINHD-1X5" device="" package3d_urn="urn:adsk.eagle:package:22469/2" value="EXTRA"/>
 <part name="TX/RX_OPT" library="pinhead" library_urn="urn:adsk.eagle:library:325" deviceset="PINHD-1X2" device="" package3d_urn="urn:adsk.eagle:package:22435/2" value="TX/RX_OPT"/>
@@
 <part name="TP18" library="testpad" library_urn="urn:adsk.eagle:library:385" deviceset="TP" device="TP10R" package3d_urn="urn:adsk.eagle:package:27959/1"/>
 <part name="TP19" library="testpad" library_urn="urn:adsk.eagle:library:385" deviceset="TP" device="TP10R" package3d_urn="urn:adsk.eagle:package:27959/1"/>
-<part name="TP20" library="testpad" library_urn="urn:adsk.eagle:library:385" deviceset="TP" device="TP10R" package3d_urn="urn:adsk.eagle:package:27959/1"/>
 <part name="GND6" library="testpad" library_urn="urn:adsk.eagle:library:385" deviceset="TP" device="TP20SQ" package3d_urn="urn:adsk.eagle:package:27980/1" value="TPTP20SQ"/>
 <part name="GND_1" library="testpad" library_urn="urn:adsk.eagle:library:385" deviceset="TP" device="TP20SQ" package3d_urn="urn:adsk.eagle:package:27980/1" value="TPTP20SQ"/>
@@
 <part name="C3" library="rcl" library_urn="urn:adsk.eagle:library:334" deviceset="C-EU" device="C0805K" package3d_urn="urn:adsk.eagle:package:23681/2" value="100n"/>
 <part name="GND7" library="supply1" library_urn="urn:adsk.eagle:library:371" deviceset="GND" device=""/>
-<part name="U$4" library="project" deviceset="RN2483" device=""/>
+<part name="U4" library="project" deviceset="RN2483" device=""/>
 <part name="GND8" library="supply1" library_urn="urn:adsk.eagle:library:371" deviceset="GND" device=""/>
 <part name="C4" library="rcl" library_urn="urn:adsk.eagle:library:334" deviceset="C-EU" device="C0603K" package3d_urn="urn:adsk.eagle:package:23680/2"/>
@@
 <part name="LORA_RX" library="SparkFun-Jumpers" deviceset="JUMPER-SMT_2_NO" device="_SILK" value="LORA_RX"/>
 <part name="LORA_TX" library="SparkFun-Jumpers" deviceset="JUMPER-SMT_2_NO" device="_SILK" value="LORA_TX"/>
+<part name="EXTRA1" library="pinhead" library_urn="urn:adsk.eagle:library:325" deviceset="PINHD-1X2" device="" package3d_urn="urn:adsk.eagle:package:22435/2" value="EXTRA"/>
 </parts>
 <sheets>
@@
 <attribute name="VALUE" x="266.7" y="-289.56" size="1.778" layer="96" font="vector" rot="R180" align="top-left"/>
 </instance>
-<instance part="LORA" gate="A" x="38.1" y="-330.2" smashed="yes">
-<attribute name="NAME" x="31.75" y="-321.945" size="1.778" layer="95"/>
-<attribute name="VALUE" x="31.75" y="-340.36" size="1.778" layer="96"/>
-</instance>
 <instance part="EXTRA" gate="A" x="0" y="-330.2" smashed="yes">
 <attribute name="NAME" x="-6.35" y="-321.945" size="1.778" layer="95"/>
@@
 <attribute name="TP_SIGNAL_NAME" x="212.09" y="-303.53" size="1.778" layer="97"/>
 </instance>
-<instance part="TP20" gate="G$1" x="170.18" y="-304.8" smashed="yes" rot="R90">
-<attribute name="NAME" x="168.91" y="-306.07" size="1.778" layer="95" rot="R90"/>
-<attribute name="TP_SIGNAL_NAME" x="171.45" y="-303.53" size="1.778" layer="97" rot="R90"/>
-</instance>
 <instance part="GND6" gate="G$1" x="365.76" y="-370.84" smashed="yes">
 <attribute name="NAME" x="364.49" y="-369.57" size="1.778" layer="95"/>
@@
 <attribute name="VALUE" x="449.58" y="-279.4" size="1.778" layer="96"/>
 </instance>
-<instance part="U$4" gate="G$1" x="515.62" y="-274.32" smashed="yes">
+<instance part="U4" gate="G$1" x="515.62" y="-274.32" smashed="yes">
 <attribute name="NAME" x="510.54" y="-260.35" size="1.778" layer="95"/>
 <attribute name="VALUE" x="510.54" y="-264.16" size="1.778" layer="96"/>
@@
 <attribute name="NAME" x="558.8" y="-281.94" size="1.778" layer="95" font="vector" rot="R180"/>
 <attribute name="VALUE" x="558.8" y="-276.86" size="1.778" layer="96" font="vector" rot="R180" align="top-left"/>
+</instance>
+<instance part="EXTRA1" gate="G$1" x="106.68" y="-358.14" smashed="yes">
+<attribute name="NAME" x="100.33" y="-352.425" size="1.778" layer="95"/>
+<attribute name="VALUE" x="100.33" y="-363.22" size="1.778" layer="96"/>
 </instance>
 </instances>
@@
 </segment>
 <segment>
-<pinref part="U$4" gate="G$1" pin="GND"/>
+<pinref part="U4" gate="G$1" pin="GND"/>
 <wire x1="538.48" y1="-292.1" x2="541.02" y2="-292.1" width="0.1524" layer="91"/>
 <pinref part="GND8" gate="1" pin="GND"/>
@@
 </segment>
 <segment>
-<pinref part="LORA" gate="A" pin="3"/>
-<wire x1="35.56" y1="-330.2" x2="20.32" y2="-330.2" width="0.1524" layer="91"/>
-<label x="20.32" y="-330.2" size="1.27" layer="95" rot="R180" xref="yes"/>
-</segment>
-<segment>
 <pinref part="LORA_RESET" gate="G$1" pin="1"/>
 <wire x1="563.88" y1="-274.32" x2="579.12" y2="-274.32" width="0.1524" layer="91"/>
 <label x="579.12" y="-274.32" size="1.778" layer="95" xref="yes"/>
-</segment>
-</net>
-<net name="SENSOR_EN" class="0">
-<segment>
-<pinref part="IC2" gate="G$1" pin="PA9"/>
-<wire x1="175.26" y1="-302.26" x2="175.26" y2="-307.34" width="0.1524" layer="91"/>
-<label x="175.26" y="-307.34" size="1.27" layer="95" rot="R270" xref="yes"/>
-</segment>
-<segment>
-<pinref part="LORA" gate="A" pin="2"/>
-<wire x1="35.56" y1="-327.66" x2="20.32" y2="-327.66" width="0.1524" layer="91"/>
-<label x="20.32" y="-327.66" size="1.27" layer="95" rot="R180" xref="yes"/>
-</segment>
-</net>
-<net name="LORA_EN" class="0">
-<segment>
-<pinref part="IC2" gate="G$1" pin="PA8"/>
-<wire x1="172.72" y1="-302.26" x2="172.72" y2="-304.8" width="0.1524" layer="91"/>
-<label x="172.72" y="-307.34" size="1.27" layer="95" rot="R270" xref="yes"/>
-<pinref part="TP20" gate="G$1" pin="TP"/>
-<wire x1="172.72" y1="-304.8" x2="172.72" y2="-307.34" width="0.1524" layer="91"/>
-<junction x="172.72" y="-304.8"/>
-</segment>
-<segment>
-<pinref part="LORA" gate="A" pin="1"/>
-<wire x1="35.56" y1="-325.12" x2="20.32" y2="-325.12" width="0.1524" layer="91"/>
-<label x="20.32" y="-325.12" size="1.27" layer="95" rot="R180" xref="yes"/>
 </segment>
 </net>
@@
 <wire x1="215.9" y1="-292.1" x2="220.98" y2="-292.1" width="0.1524" layer="91"/>
 <junction x="215.9" y="-292.1"/>
-</segment>
-<segment>
-<pinref part="LORA" gate="A" pin="5"/>
-<wire x1="35.56" y1="-335.28" x2="20.32" y2="-335.28" width="0.1524" layer="91"/>
-<label x="20.32" y="-335.28" size="1.27" layer="95" rot="R180" xref="yes"/>
 </segment>
 <segment>
@@
 <pinref part="TP19" gate="G$1" pin="TP"/>
 <junction x="210.82" y="-304.8"/>
-</segment>
-<segment>
-<wire x1="35.56" y1="-332.74" x2="20.32" y2="-332.74" width="0.1524" layer="91"/>
-<pinref part="LORA" gate="A" pin="4"/>
-<label x="20.32" y="-332.74" size="1.27" layer="95" rot="R180" xref="yes"/>
 </segment>
 <segment>
@@
 <segment>
 <pinref part="C4" gate="G$1" pin="2"/>
-<pinref part="U$4" gate="G$1" pin="RFH"/>
+<pinref part="U4" gate="G$1" pin="RFH"/>
 <wire x1="551.18" y1="-269.24" x2="548.64" y2="-269.24" width="0.1524" layer="91"/>
 <wire x1="548.64" y1="-269.24" x2="538.48" y2="-269.24" width="0.1524" layer="91"/>
@@
 <net name="N$6" class="0">
 <segment>
-<pinref part="U$4" gate="G$1" pin="UART_RX"/>
+<pinref part="U4" gate="G$1" pin="UART_RX"/>
 <wire x1="538.48" y1="-276.86" x2="571.5" y2="-276.86" width="0.1524" layer="91"/>
 <pinref part="LORA_RX" gate="G$1" pin="2"/>
@@
 <net name="N$7" class="0">
 <segment>
-<pinref part="U$4" gate="G$1" pin="UART_TX"/>
+<pinref part="U4" gate="G$1" pin="UART_TX"/>
 <wire x1="538.48" y1="-279.4" x2="551.18" y2="-279.4" width="0.1524" layer="91"/>
 <pinref part="LORA_TX" gate="G$1" pin="2"/>
@@
 <net name="N$8" class="0">
 <segment>
-<pinref part="U$4" gate="G$1" pin="RESET°"/>
+<pinref part="U4" gate="G$1" pin="RESET°"/>
 <wire x1="538.48" y1="-274.32" x2="553.72" y2="-274.32" width="0.1524" layer="91"/>
 <pinref part="LORA_RESET" gate="G$1" pin="2"/>
@@
 </segment>
 <segment>
-<pinref part="U$4" gate="G$1" pin="VDD"/>
+<pinref part="U4" gate="G$1" pin="VDD"/>
 <wire x1="538.48" y1="-289.56" x2="558.8" y2="-289.56" width="0.1524" layer="91"/>
 <pinref part="LORA_VDD" gate="G$1" pin="2"/>
@@
 </segment>
 </net>
+<net name="PA8" class="0">
+<segment>
+<pinref part="IC2" gate="G$1" pin="PA8"/>
+<wire x1="172.72" y1="-302.26" x2="172.72" y2="-307.34" width="0.1524" layer="91"/>
+<label x="172.72" y="-307.34" size="1.27" layer="95" rot="R270" xref="yes"/>
+</segment>
+<segment>
+<pinref part="EXTRA1" gate="G$1" pin="1"/>
+<wire x1="104.14" y1="-355.6" x2="93.98" y2="-355.6" width="0.1524" layer="91"/>
+<label x="93.98" y="-355.6" size="1.27" layer="95" rot="R180" xref="yes"/>
+</segment>
+</net>
+<net name="PA9" class="0">
+<segment>
+<pinref part="IC2" gate="G$1" pin="PA9"/>
+<wire x1="175.26" y1="-302.26" x2="175.26" y2="-307.34" width="0.1524" layer="91"/>
+<label x="175.26" y="-307.34" size="1.27" layer="95" rot="R270" xref="yes"/>
+</segment>
+<segment>
+<pinref part="EXTRA1" gate="G$1" pin="2"/>
+<wire x1="104.14" y1="-358.14" x2="93.98" y2="-358.14" width="0.1524" layer="91"/>
+<label x="93.98" y="-358.14" size="1.27" layer="95" rot="R180" xref="yes"/>
+</segment>
+</net>

Commit message: PCB's DONE! :100:
Parts:
- EXTRA: device pinhead:PINHD-1X5 -> pinhead:PINHD-1X4
Connections:
- net PC9: now also EXTRA.1; no longer EXTRA.2
- net PE13: now also EXTRA.4; no longer EXTRA.5
- net PF3: now also EXTRA.2; no longer EXTRA.3
- net PF5: now also EXTRA.3; no longer EXTRA.4
Changed lines of the file:
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@@
 <part name="BATT_V" library="SparkFun-Jumpers" deviceset="JUMPER-SMT_2_NO" device="_SILK" value="BATT_V"/>
 <part name="SOLAR_V" library="SparkFun-Jumpers" deviceset="JUMPER-SMT_2_NO" device="_SILK" value="SOLAR_V"/>
-<part name="EXTRA" library="pinhead" library_urn="urn:adsk.eagle:library:325" deviceset="PINHD-1X5" device="" package3d_urn="urn:adsk.eagle:package:22469/2" value="EXTRA"/>
 <part name="TX/RX_OPT" library="pinhead" library_urn="urn:adsk.eagle:library:325" deviceset="PINHD-1X2" device="" package3d_urn="urn:adsk.eagle:package:22435/2" value="TX/RX_OPT"/>
 <part name="DBG_OPT" library="pinhead" library_urn="urn:adsk.eagle:library:325" deviceset="PINHD-1X2" device="" package3d_urn="urn:adsk.eagle:package:22435/2" value="DBG_OPT"/>
@@
 <part name="LORA_TX" library="SparkFun-Jumpers" deviceset="JUMPER-SMT_2_NO" device="_SILK" value="LORA_TX"/>
 <part name="EXTRA1" library="pinhead" library_urn="urn:adsk.eagle:library:325" deviceset="PINHD-1X2" device="" package3d_urn="urn:adsk.eagle:package:22435/2" value="EXTRA"/>
+<part name="EXTRA" library="pinhead" library_urn="urn:adsk.eagle:library:325" deviceset="PINHD-1X4" device="" package3d_urn="urn:adsk.eagle:package:22407/2" value="EXTRA"/>
 </parts>
 <sheets>
@@
 <attribute name="VALUE" x="266.7" y="-289.56" size="1.778" layer="96" font="vector" rot="R180" align="top-left"/>
 </instance>
-<instance part="EXTRA" gate="A" x="0" y="-330.2" smashed="yes">
-<attribute name="NAME" x="-6.35" y="-321.945" size="1.778" layer="95"/>
-<attribute name="VALUE" x="-6.35" y="-340.36" size="1.778" layer="96"/>
-</instance>
 <instance part="TX/RX_OPT" gate="G$1" x="-2.54" y="-299.72" smashed="yes">
 <attribute name="NAME" x="-8.89" y="-294.005" size="1.778" layer="95"/>
@@
 <attribute name="NAME" x="100.33" y="-352.425" size="1.778" layer="95"/>
 <attribute name="VALUE" x="100.33" y="-363.22" size="1.778" layer="96"/>
+</instance>
+<instance part="EXTRA" gate="A" x="0" y="-332.74" smashed="yes">
+<attribute name="NAME" x="-6.35" y="-324.485" size="1.778" layer="95"/>
+<attribute name="VALUE" x="-6.35" y="-340.36" size="1.778" layer="96"/>
 </instance>
 </instances>
@@
 <label x="-12.7" y="-335.28" size="1.27" layer="95" rot="R180" xref="yes"/>
 <wire x1="-12.7" y1="-335.28" x2="-2.54" y2="-335.28" width="0.1524" layer="91"/>
-<pinref part="EXTRA" gate="A" pin="5"/>
+<pinref part="EXTRA" gate="A" pin="4"/>
 </segment>
 </net>
@@
 <label x="-12.7" y="-327.66" size="1.27" layer="95" rot="R180" xref="yes"/>
 <wire x1="-2.54" y1="-327.66" x2="-12.7" y2="-327.66" width="0.1524" layer="91"/>
-<pinref part="EXTRA" gate="A" pin="2"/>
+<pinref part="EXTRA" gate="A" pin="1"/>
 </segment>
 </net>
@@
 <wire x1="-2.54" y1="-330.2" x2="-12.7" y2="-330.2" width="0.1524" layer="91"/>
 <label x="-12.7" y="-330.2" size="1.27" layer="95" rot="R180" xref="yes"/>
-<pinref part="EXTRA" gate="A" pin="3"/>
+<pinref part="EXTRA" gate="A" pin="2"/>
 </segment>
 </net>
@@
 <label x="-12.7" y="-332.74" size="1.27" layer="95" rot="R180" xref="yes"/>
 <wire x1="-2.54" y1="-332.74" x2="-12.7" y2="-332.74" width="0.1524" layer="91"/>
-<pinref part="EXTRA" gate="A" pin="4"/>
+<pinref part="EXTRA" gate="A" pin="3"/>
 </segment>
 </net>
@@
 </sheet>
 </sheets>
+<errors>
+</errors>
 </schematic>
 </drawing>
